Commit message: Adding final urdf/gazebo robot

File: ros2_ws/src/my_robot_description/urdf/camera.xacro (robot description, xacro)
@@ -7,8 +7,8 @@
   <link name="camera_link">
     <visual>
-        <geometry>
-          <box size="${camera_length} ${camera_width} ${camera_height}" />
-          </geometry>
-        <material name="gray" />
+      <geometry>
+        <box size="${camera_length} ${camera_width} ${camera_height}" />
+      </geometry>
+      <material name="gray" />
     </visual>
     <collision>
@@ -16,5 +16,5 @@
     </collision>
     <xacro:box_inertia m="0.1" l="${camera_length}" w="${camera_width}" h="${camera_height}"
-      xyz="0 0 0" rpy="0 0 0"/>
+      xyz="0 0 0" rpy="0 0 0" />
   </link>
   <joint name="base_camera_joint" type="fixed">
@@ -23,6 +23,21 @@
     <origin xyz="${(base_length + camera_length) / 2.0} 0 ${base_height / 2.0}" rpy="0 0 0" />
   </joint>
+  <link name="camera_link_optical">
+  </link>
+  <joint name="camera_optical_joint" type="fixed">
+    <origin xyz="0 0 0" rpy="${-pi/2} 0 ${-pi/2}" />
+    <parent link="camera_link" />
+    <child link="camera_link_optical" />
+  </joint>
   <gazebo reference="camera_link">
     <material>Gazebo/Red</material>
-    </gazebo>
+    <sensor name="camera_sensor" type="camera">
+      <pose>0 0 0 0 0 0</pose>
+      <visualize>true</visualize>
+      <update_rate>10.0</update_rate>
+      <plugin name="camera_controller" filename="libgazebo_ros_camera.so">
+        <frame_name>camera_link_optical</frame_name>
+      </plugin>
+    </sensor>
+  </gazebo>
 </robot>

File: ros2_ws/src/my_robot_description/urdf/common_properties.xacro (robot description, xacro)
@@ -10,4 +10,10 @@
   <material name="gray">
     <color rgba="0.5 0.5 0.5 1" />
+  </material>
+  <material name="orange">
+    <color rgba="1 0.64 0 1" />
+  </material>
+  <material name="yellow">
+    <color rgba="1 1 0 1" />
   </material>
   <xacro:macro name="box_inertia" params="m l w h xyz rpy">

File: ros2_ws/src/my_robot_description/urdf/my_robot.urdf.xacro (robot description, xacro)
@@ -5,4 +5,11 @@
   <xacro:include filename="mobile_base.xacro" />
   <xacro:include filename="mobile_base_gazebo.xacro" />
-  <xacro:include filename="camera.xacro" />
+  <xacro:include filename="arm.xacro" />
+  <xacro:include filename="arm_gazebo.xacro" />
+  <!-- <xacro:include filename="camera.xacro" /> -->
+  <joint name="mobile_base_arm_joint" type="fixed">
+    <parent link="base_link" />
+    <child link="arm_base_link" />
+    <origin xyz="${base_length  / 4.0} 0 ${base_height}" rpy="0 0 0" />
+  </joint>
 </robot>
